File: ergo33/ergo33.sch (KiCad schematic (older format))
At the start: 112 parts, among them SW1 SW_Push, SW46 Rotary_Encoder_Switch, U1 ATmega32U4-AU, U2 USBLC6-2SC6, Y1 16MHz

Commit message: Add external light PCB
Parts:
- added CExt1, CExt2, CExt3, CExt4: 0,1uF, Capacitor_SMD:C_0805_2012Metric_Pad1.15x1.40mm_HandSolder, symbol Device:C_Small
- added JExt1: Conn_01x03, Connector_PinHeader_2.54mm:PinHeader_1x03_P2.54mm_Vertical, symbol Connector_Generic:Conn_01x03
- added LEDExt1, LEDExt2, LEDExt3, LEDExt4: WS2812B, LED_SMD:LED_WS2812B_PLCC4_5.0x5.0mm_P3.2mm, symbol LED:WS2812B
- C1, C10, C11, C12, C13, C14, C15, C16, C17, C18, C19, C2, C20, C3, C4, C5, C6, C7, C8, C9: footprint Capacitor_SMD:C_0805_2012Metric -> Capacitor_SMD:C_0805_2012Metric_Pad1.15x1.40mm_HandSolder
- F1: footprint Fuse:Fuse_1206_3216Metric -> Fuse:Fuse_1206_3216Metric_Pad1.42x1.75mm_HandSolder
- R1, R2, R3, R4, R5, R6: footprint Resistor_SMD:R_0805_2012Metric -> Resistor_SMD:R_0805_2012Metric_Pad1.15x1.40mm_HandSolder
- Y1: footprint Crystal:Crystal_SMD_3225-4Pin_3.2x2.5mm -> Crystal:Crystal_SMD_3225-4Pin_3.2x2.5mm_HandSoldering
Connections:
- net +5V: now also JLED1.3 (Pin_3); no longer JLED1.1 (Pin_1)
- net GND: now also JLED1.1 (Pin_1); no longer JLED1.3 (Pin_3)
- new net: JExt1.2 (Pin_2), LEDExt1.4 (DIN)
- new net: LEDExt1.2 (DOUT), LEDExt2.4 (DIN)
- new net: LEDExt2.2 (DOUT), LEDExt3.4 (DIN)
- new net: LEDExt3.2 (DOUT), LEDExt4.4 (DIN)
- new net 5VExt: CExt1.1, CExt2.1, CExt3.1, CExt4.1, JExt1.3 (Pin_3), LEDExt1.1 (VDD), LEDExt2.1 (VDD), LEDExt3.1 (VDD), LEDExt4.1 (VDD)
- new net GNDExt: CExt1.2, CExt2.2, CExt3.2, CExt4.2, JExt1.1 (Pin_1), LEDExt1.3 (VSS), LEDExt2.3 (VSS), LEDExt3.3 (VSS), LEDExt4.3 (VSS)
- no-connect marks 2 -> 14
Other:
- moved on the sheet: C20, F1, R5, R6, U2, USB1
