File: ergo33/ergo33.kicad_pcb (KiCad board)
At the start: 2 copper layers, 173.8 x 121.8 mm, 135 parts, among them M1 MountingHole_2.2mm_M2_ISO7380, M2 MountingHole_2.2mm_M2_ISO7380, SW1 SW_Push, SW46 Rotary_Encoder_Switch, U1 ATmega32U4-AU, U2 USBLC6-2SC6, Y1 16MHz

Commit message: ergo33: Panelize maybe?
Parts:
- added REF**: breakaway-mousebites, random-keyboard-parts:breakaway-mousebites, F.Cu at (56.2, 114.7)
- added REF**: breakaway-mousebites, random-keyboard-parts:breakaway-mousebites, F.Cu at (56.2, 116.7)
- added REF**: breakaway-mousebites, random-keyboard-parts:breakaway-mousebites, F.Cu at (31.8, 114.7)
- added REF**: breakaway-mousebites, random-keyboard-parts:breakaway-mousebites, F.Cu at (31.8, 116.7)
Other:
- outline, holes or cut-outs redrawn
Changed lines of the file:
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@@
   (general
     (thickness 1.6)
-    (drawings 28)
+    (drawings 44)
     (tracks 996)
     (zones 0)
-    (modules 135)
+    (modules 139)
     (nets 83)
   )
@@
     (38 B.Mask user)
     (39 F.Mask user)
-    (40 Dwgs.User user)
+    (40 Dwgs.User user hide)
     (41 Cmts.User user)
     (42 Eco1.User user)
@@
     (44 Edge.Cuts user)
     (45 Margin user)
-    (46 B.CrtYd user)
-    (47 F.CrtYd user)
+    (46 B.CrtYd user hide)
+    (47 F.CrtYd user hide)
     (48 B.Fab user)
     (49 F.Fab user)
@@
     (visible_elements 7FFFFFFF)
     (pcbplotparams
-      (layerselection 0x010fc_ffffffff)
-      (usegerberextensions false)
-      (usegerberattributes true)
-      (usegerberadvancedattributes true)
-      (creategerberjobfile true)
+      (layerselection 0x010f0_ffffffff)
+      (usegerberextensions true)
+      (usegerberattributes false)
+      (usegerberadvancedattributes false)
+      (creategerberjobfile false)
       (excludeedgelayer true)
       (linewidth 0.100000)
@@
       (plotinvisibletext false)
       (padsonsilk false)
-      (subtractmaskfromsilk false)
+      (subtractmaskfromsilk true)
       (outputformat 1)
       (mirror false)
-      (drillshape 1)
+      (drillshape 0)
       (scaleselection 1)
-      (outputdirectory ""))
+      (outputdirectory "./gerber"))
   )
   (net 0 "")
@@
     (add_net VBUS)
   )
+  (module random-keyboard-parts:breakaway-mousebites (layer F.Cu)
+    (at 56.2 114.7)
+    (attr virtual)
+    (fp_text reference REF** (at 0 -1.524) (layer Dwgs.User)
+      (effects (font (size 1 1) (thickness 0.15)))
+    )
+    (fp_text value breakaway-mousebites (at 0 0.762) (layer Dwgs.User)
+      (effects (font (size 1 1) (thickness 0.15)))
+    )
+    (fp_line (start -2.794 0) (end 2.794 0) (layer Dwgs.User) (width 0.15))
+    (fp_line (start 0.254 0) (end -0.254 0) (layer B.CrtYd) (width 0.15))
+    (fp_line (start -1.016 0) (end -1.524 0) (layer B.CrtYd) (width 0.15))
+    (fp_line (start -2.286 0) (end -2.794 0) (layer B.CrtYd) (width 0.15))
+    (fp_line (start 1.016 0) (end 1.524 0) (layer B.CrtYd) (width 0.15))
+    (fp_line (start 2.286 0) (end 2.794 0) (layer B.CrtYd) (width 0.15))
+    (pad "" np_thru_hole circle (at 0 -0.254) (size 0.7874 0.7874) (drill 0.7874) (layers *.Cu *.Mask))
+    (pad "" np_thru_hole circle (at 1.27 -0.254) (size 0.7874 0.7874) (drill 0.7874) (layers *.Cu *.Mask))
+    (pad "" np_thru_hole circle (at 2.54 -0.254) (size 0.7874 0.7874) (drill 0.7874) (layers *.Cu *.Mask))
+    (pad "" np_thru_hole circle (at -1.27 -0.254) (size 0.7874 0.7874) (drill 0.7874) (layers *.Cu *.Mask))
+    (pad "" np_thru_hole circle (at -2.54 -0.254) (size 0.7874 0.7874) (drill 0.7874) (layers *.Cu *.Mask))
+  )
+  (module random-keyboard-parts:breakaway-mousebites (layer F.Cu)
+    (at 56.2 116.654)
+    (attr virtual)
+    (fp_text reference REF** (at 0 -1.524) (layer Dwgs.User)
+      (effects (font (size 1 1) (thickness 0.15)))
+    )
+    (fp_text value breakaway-mousebites (at 0 0.762) (layer Dwgs.User)
+      (effects (font (size 1 1) (thickness 0.15)))
+    )
+    (fp_line (start -2.794 0) (end 2.794 0) (layer Dwgs.User) (width 0.15))
+    (fp_line (start 0.254 0) (end -0.254 0) (layer B.CrtYd) (width 0.15))
+    (fp_line (start -1.016 0) (end -1.524 0) (layer B.CrtYd) (width 0.15))
+    (fp_line (start -2.286 0) (end -2.794 0) (layer B.CrtYd) (width 0.15))
+    (fp_line (start 1.016 0) (end 1.524 0) (layer B.CrtYd) (width 0.15))
+    (fp_line (start 2.286 0) (end 2.794 0) (layer B.CrtYd) (width 0.15))
+    (pad "" np_thru_hole circle (at 0 -0.254) (size 0.7874 0.7874) (drill 0.7874) (layers *.Cu *.Mask))
+    (pad "" np_thru_hole circle (at 1.27 -0.254) (size 0.7874 0.7874) (drill 0.7874) (layers *.Cu *.Mask))
+    (pad "" np_thru_hole circle (at 2.54 -0.254) (size 0.7874 0.7874) (drill 0.7874) (layers *.Cu *.Mask))
+    (pad "" np_thru_hole circle (at -1.27 -0.254) (size 0.7874 0.7874) (drill 0.7874) (layers *.Cu *.Mask))
+    (pad "" np_thru_hole circle (at -2.54 -0.254) (size 0.7874 0.7874) (drill 0.7874) (layers *.Cu *.Mask))
+  )
+  (module random-keyboard-parts:breakaway-mousebites (layer F.Cu)
+    (at 31.8 114.7)
+    (attr virtual)
+    (fp_text reference REF** (at 0 -1.524) (layer Dwgs.User)
+      (effects (font (size 1 1) (thickness 0.15)))
+    )
+    (fp_text value breakaway-mousebites (at 0 0.762) (layer Dwgs.User)
+      (effects (font (size 1 1) (thickness 0.15)))
+    )
+    (fp_line (start -2.794 0) (end 2.794 0) (layer Dwgs.User) (width 0.15))
+    (fp_line (start 0.254 0) (end -0.254 0) (layer B.CrtYd) (width 0.15))
+    (fp_line (start -1.016 0) (end -1.524 0) (layer B.CrtYd) (width 0.15))
+    (fp_line (start -2.286 0) (end -2.794 0) (layer B.CrtYd) (width 0.15))
+    (fp_line (start 1.016 0) (end 1.524 0) (layer B.CrtYd) (width 0.15))
+    (fp_line (start 2.286 0) (end 2.794 0) (layer B.CrtYd) (width 0.15))
+    (pad "" np_thru_hole circle (at 0 -0.254) (size 0.7874 0.7874) (drill 0.7874) (layers *.Cu *.Mask))
+    (pad "" np_thru_hole circle (at 1.27 -0.254) (size 0.7874 0.7874) (drill 0.7874) (layers *.Cu *.Mask))
+    (pad "" np_thru_hole circle (at 2.54 -0.254) (size 0.7874 0.7874) (drill 0.7874) (layers *.Cu *.Mask))
+    (pad "" np_thru_hole circle (at -1.27 -0.254) (size 0.7874 0.7874) (drill 0.7874) (layers *.Cu *.Mask))
+    (pad "" np_thru_hole circle (at -2.54 -0.254) (size 0.7874 0.7874) (drill 0.7874) (layers *.Cu *.Mask))
+  )
+  (module random-keyboard-parts:breakaway-mousebites (layer F.Cu)
+    (at 31.8 116.654)
+    (attr virtual)
+    (fp_text reference REF** (at 0 -1.524) (layer Dwgs.User)
+      (effects (font (size 1 1) (thickness 0.15)))
+    )
+    (fp_text value breakaway-mousebites (at 0 0.762) (layer Dwgs.User)
+      (effects (font (size 1 1) (thickness 0.15)))
+    )
+    (fp_line (start -2.794 0) (end 2.794 0) (layer Dwgs.User) (width 0.15))
+    (fp_line (start 0.254 0) (end -0.254 0) (layer B.CrtYd) (width 0.15))
+    (fp_line (start -1.016 0) (end -1.524 0) (layer B.CrtYd) (width 0.15))
+    (fp_line (start -2.286 0) (end -2.794 0) (layer B.CrtYd) (width 0.15))
+    (fp_line (start 1.016 0) (end 1.524 0) (layer B.CrtYd) (width 0.15))
+    (fp_line (start 2.286 0) (end 2.794 0) (layer B.CrtYd) (width 0.15))
+    (pad "" np_thru_hole circle (at -2.54 -0.254) (size 0.7874 0.7874) (drill 0.7874) (layers *.Cu *.Mask))
+    (pad "" np_thru_hole circle (at -1.27 -0.254) (size 0.7874 0.7874) (drill 0.7874) (layers *.Cu *.Mask))
+    (pad "" np_thru_hole circle (at 2.54 -0.254) (size 0.7874 0.7874) (drill 0.7874) (layers *.Cu *.Mask))
+    (pad "" np_thru_hole circle (at 1.27 -0.254) (size 0.7874 0.7874) (drill 0.7874) (layers *.Cu *.Mask))
+    (pad "" np_thru_hole circle (at 0 -0.254) (size 0.7874 0.7874) (drill 0.7874) (layers *.Cu *.Mask))
+  )
   (module LED_SMD:LED_WS2812B_PLCC4_5.0x5.0mm_P3.2mm (layer F.Cu)
     (at 38.31 124.27 180)
@@
     )
   )
+  (gr_line (start 59.5 115.01) (end 59.5 115.79) (layer Edge.Cuts) (width 0.2))
+  (gr_arc (start 60.5 115.79) (end 59.5 115.79) (angle -90) (layer Edge.Cuts) (width 0.2))
+  (gr_arc (start 60.5 115.01) (end 60.5 114.01) (angle -90) (layer Edge.Cuts) (width 0.2))
+  (gr_line (start 67.909999 116.79) (end 60.5 116.79) (layer Edge.Cuts) (width 0.2))
+  (gr_line (start 60.882464 114.01) (end 60.5 114.01) (layer Edge.Cuts) (width 0.2))
+  (gr_line (start 53 115.01) (end 53 115.79) (layer Edge.Cuts) (width 0.2))
+  (gr_arc (start 52 115.01) (end 53 115.01) (angle -90) (layer Edge.Cuts) (width 0.2))
+  (gr_arc (start 52 115.79) (end 52 116.79) (angle -90) (layer Edge.Cuts) (width 0.2))
+  (gr_line (start 35 115.79) (end 35 115.01) (layer Edge.Cuts) (width 0.2))
+  (gr_arc (start 36 115.79) (end 35 115.79) (angle -90) (layer Edge.Cuts) (width 0.2))
+  (gr_line (start 28.5 115.79) (end 28.5 115.01) (layer Edge.Cuts) (width 0.2))
+  (gr_arc (start 27.5 115.79) (end 27.5 116.79) (angle -90) (layer Edge.Cuts) (width 0.2))
+  (gr_line (start 26.334451 114.01) (end 27.5 114.01) (layer Edge.Cuts) (width 0.2))
+  (gr_line (start 26.81 116.79) (end 27.5 116.79) (layer Edge.Cuts) (width 0.2))
+  (gr_arc (start 27.5 115.01) (end 28.5 115.01) (angle -90) (layer Edge.Cuts) (width 0.2))
+  (gr_arc (start 36 115.01) (end 36 114.01) (angle -90) (layer Edge.Cuts) (width 0.2))
+  (gr_line (start 36 116.79) (end 52 116.79) (layer Edge.Cuts) (width 0.2))
+  (gr_line (start 36 114.01) (end 52 114.01) (layer Edge.Cuts) (width 0.2))
   (gr_text Layer (at 56.11 131.97 270) (layer F.SilkS)
     (effects (font (size 2 2) (thickness 0.3)))
@@
   )
   (gr_arc (start 26.810001 137.555961) (end 23.810001 137.555961) (angle -94.3) (layer Edge.Cuts) (width 0.2))
-  (gr_line (start 26.81 116.79) (end 67.910001 116.79) (layer Edge.Cuts) (width 0.2))
   (gr_line (start 27.034937 140.547516) (end 68.134937 137.457192) (layer Edge.Cuts) (width 0.2))
   (gr_line (start 23.810001 119.79) (end 23.810001 137.555961) (layer Edge.Cuts) (width 0.2))
@@
   (gr_line (start 23.81445 21.28) (end 23.81445 111.490001) (layer Edge.Cuts) (width 0.2))
   (gr_line (start 157.543918 28.11) (end 185.48 28.11) (layer Edge.Cuts) (width 0.2))
-  (gr_line (start 26.334449 114.01) (end 60.882464 114.01) (layer Edge.Cuts) (width 0.2))
   (gr_line (start 193.207804 35.273874) (end 197.60717 93.277415) (layer Edge.Cuts) (width 0.2))
   (gr_line (start 167.126474 133.581012) (end 191.797626 108.94109) (layer Edge.Cuts) (width 0.2))
@@
     (polygon
       (pts
-        (xy 196.8 27.4) (xy 201 101.5) (xy 171.8 144.1) (xy 62.4 114.3) (xy 20.3 115)
+        (xy 196.8 27.4) (xy 201 101.5) (xy 171.8 144.1) (xy 60.8 113.4) (xy 22.7 113.4)
         (xy 14.7 20) (xy 23.2 16.5) (xy 82.2 16.5)
       )
@@
     (polygon
       (pts
-        (xy 68.4 116.6) (xy 70.9 117.7) (xy 72.1 137.6) (xy 23 141.5) (xy 23.4 116)
+        (xy 68.5 117.4) (xy 70.9 117.7) (xy 72.1 137.6) (xy 23 141.5) (xy 23.4 117.4)
       )
     )

Commit message: Ergo33: add graphics
Parts:
- added G***: LOGO, tunks-parts:Logo_Ergo33_33.1x9.0mm, B.Cu at (90.7, 111.1)
- added G***: LOGO, tunks-parts:Logo_Kulmajaba_20.0x11.3mm, F.Cu at (86.3, 112.4)
- added G***: LOGO, tunks-parts:Text_Layer_7.3x3.0mm, F.Cu at (56.1, 131.7)
- added G***: LOGO, tunks-parts:Text_Mode_7.6x3.1mm, F.Cu at (65.0, 131.8)
Other:
- board text added: "If you can read this, your keypad probably doesn't work"
- board text added: "JLCJLCJLCJLC"
- board text removed: "Layer"
- board text removed: "Mode"

Commit message: Ergo33: depanelize :(
Parts:
- removed CExt1, CExt2, CExt3, CExt4: 0,1uF, Capacitor_SMD:C_0805_2012Metric_Pad1.15x1.40mm_HandSolder
- removed the G*** at (56.1, 131.7)
- removed the G*** at (65.0, 131.8)
- removed JExt1: Conn_01x03, Connector_PinHeader_2.54mm:PinHeader_1x03_P2.54mm_Vertical
- removed LEDExt1, LEDExt2, LEDExt3, LEDExt4: WS2812B, LED_SMD:LED_WS2812B_PLCC4_5.0x5.0mm_P3.2mm
- removed M1, M2: MountingHole_2.2mm_M2_ISO7380, MountingHole:MountingHole_2.2mm_M2_ISO7380
- removed the REF** at (56.2, 114.7)
- removed the REF** at (56.2, 116.7)
- removed the REF** at (31.8, 114.7)
- removed the REF** at (31.8, 116.7)
Routing:
- net 5VExt: track 73.8 -> 0.00 mm
- net Net-(JExt1-Pad2): track 9.91 -> 0.00 mm
- net Net-(LEDExt2-Pad2): track 5.33 -> 0.00 mm
- net Net-(LEDExt3-Pad2): track 5.33 -> 0.00 mm
- net Net-(LEDExt1-Pad2): track 5.32 -> 0.00 mm
- removed copper zone on F.Cu, net GNDExt
Other:
- board size 173.8 x 121.8 mm -> 173.8 x 117.1 mm

Commit message: Change a few cap values
Parts:
- C1, C2: value 22pF -> 16pF
- C20: value 0.1uF -> 0,1uF
- SW46: value Rotary_Encoder_Switch -> EC11_Rotary_Encoder
Connections:
- net RD+ renamed Net-(R3-Pad1)
- net RD- renamed Net-(R2-Pad1)

Commit message: Ergo33: rev2
Parts:
- removed the C20 at (173.6, 44.3)
- removed the C4 at (187.6, 55.2)
- removed the C7 at (177.7, 50.9)
- removed the R2 at (168.5, 51.0)
- removed the R3 at (171.8, 51.0)
- added C10: 16pF, Capacitor_SMD:C_0805_2012Metric_Pad1.15x1.40mm_HandSolder, B.Cu at (189.7, 62.2)
- added C3: 10uF, Capacitor_SMD:C_0805_2012Metric_Pad1.15x1.40mm_HandSolder, B.Cu at (183.2, 76.5)
- added C5: 0,1uF, Capacitor_SMD:C_0805_2012Metric_Pad1.15x1.40mm_HandSolder, B.Cu at (183.9, 60.3)
- added C9: 16pF, Capacitor_SMD:C_0805_2012Metric_Pad1.15x1.40mm_HandSolder, B.Cu at (190.2, 68.7)
- added R4: 22, Resistor_SMD:R_0805_2012Metric_Pad1.15x1.40mm_HandSolder, B.Cu at (172.3, 55.0)
- added R5: 22, Resistor_SMD:R_0805_2012Metric_Pad1.15x1.40mm_HandSolder, B.Cu at (169.6, 55.0)
- C1: value 16pF -> 0,1uF
- C2: value 16pF -> 10uF
- G***: footprint tunks-parts:Logo_Ergo33_33.1x9.0mm -> tunks-parts:Logo_Ergo33_rev2_33.1x9.0mm
- JP1: value SolderJumper_3_Bridged12 -> SolderJumper_3_Open; footprint Jumper:SolderJumper-3_P1.3mm_Bridged2Bar12_Pad1.0x1.5mm_NumberLabels -> Jumper:SolderJumper-3_P1.3mm_Open_Pad1.0x1.5mm_NumberLabels
- REF** (x12): value MountingHole_2.2mm_M2_ISO7380_Pad_Courtyard -> M2
- moved C1 35.1 mm to (168.2, 40.9), turned to 0 degrees
- moved C2 12.1 mm to (179.5, 51.4), turned to 90 degrees
- moved C11 5.80 mm to (189.4, 45.2), turned to 90 degrees
- moved SW1 3.42 mm to (184.6, 43.1)
- moved JP1 3.24 mm to (170.9, 80.9)
- moved C4 2.80 mm to (165.6, 61.3)
- moved U2 2.31 mm to (170.9, 45.5)
- moved R6 2.25 mm to (181.2, 56.0)
- moved F1 2.12 mm to (175.2, 47.0)
- moved C7 1.40 mm to (177.7, 56.0), turned to 90 degrees
- moved Y1 0.91 mm to (187.0, 65.4)
- moved C8 0.89 mm to (175.0, 56.0)
- moved C6 0.54 mm to (179.5, 75.5)
- moved C21 0.10 mm to (159.2, 80.4)
- renumbered C19 to C11, C9 to C12, C10 to C13, C11 to C14, C12 to C15, C13 to C16, C14 to C17, C15 to C18, C16 to C19, C17 to C20, C18 to C21, C3 to C4, C5 to C6, C6 to C7, R5 to R1, R6 to R2, R4 to R3, R1 to R6
Connections:
- C1 pad 2: Net-(C1-Pad2) -> VBUS
- C2 pad 1: GND -> +5V
- C2 pad 2: Net-(C2-Pad2) -> GND
- U1 pad 16: Net-(C2-Pad2) -> Net-(C10-Pad2)
- U1 pad 17: Net-(C1-Pad2) -> Net-(C9-Pad2)
- Y1 pad 1: Net-(C1-Pad2) -> Net-(C9-Pad2)
- Y1 pad 3: Net-(C2-Pad2) -> Net-(C10-Pad2)
Routing:
- net +5V: track 494.1 -> 457.2 mm
- net Net-(C2-Pad2): track 12.8 -> 0.00 mm
- net Net-(C11-Pad1): track 35.9 -> 23.6 mm, vias 2 -> 0
- net Net-(C1-Pad2): track 11.6 -> 0.00 mm
- net Net-(C9-Pad2): track 0.00 -> 10.2 mm
- net Net-(C10-Pad2): track 0.00 -> 10.0 mm
- net LEDS: track 16.8 -> 12.2 mm
- net Net-(R4-Pad1): track 10.3 -> 5.78 mm
- net Net-(R5-Pad1): track 10.2 -> 5.77 mm
- net ROW4: track 205.4 -> 202.2 mm
- net VBUS: track 24.8 -> 27.8 mm
- net DBUS+: track 12.4 -> 14.6 mm
- net D-: track 5.89 -> 7.96 mm
- net D+: track 5.94 -> 7.96 mm
- net GND: track 176.4 -> 178.0 mm, vias 31 -> 129
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- added copper zone on B.Cu, net GND

Commit message: Ergo33: Change logo to v1.1
Parts:
- G***: footprint tunks-parts:Logo_Ergo33_rev2_33.1x9.0mm -> tunks-parts:Logo_Ergo33_v2.0_33.1x9.0mm
