File: ergo33-led-board/ergo33_led_board.kicad_pcb (KiCad board)
At the start: 2 copper layers, 47.1 x 23.8 mm, 13 parts, among them M1 MountingHole_2.2mm_M2_ISO7380, M2 MountingHole_2.2mm_M2_ISO7380

Commit message: Ergo33: update LED PCB gerbers
Other:
- board text added: "JLCJLCJLCJLC"
